File: K_IO_brd.kicad_pcb (KiCad board)
At the start: 2 copper layers, 100 x 100 mm, 105 parts, among them J1 Conn from SDR J1, J10 To Andromeda J7, J11 PTT Out, J12 PTT Int, J13 SPKR Mute, J14 Jack_in/out, J15 to Andromeda J2, J18 Conn_01x02_Socket, J19 To SDR, J2 ACC Out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

Commit message: minor changes
Parts:
- removed C16, C21, C24, C25, C27: 10n, Capacitor_SMD:C_0805_2012Metric_Pad1.18x1.45mm_HandSolder
- removed FB12, FB14, FB15: fb0805, Inductor_SMD:L_0805_2012Metric_Pad1.15x1.40mm_HandSolder
- removed J3: ATU Int, Connector_Molex:Molex_KK-254_AE-6410-03A_1x03_P2.54mm_Vertical
- removed J8: Tune Ext ATU, Connector_Molex:Molex_KK-254_AE-6410-04A_1x04_P2.54mm_Vertical
- moved G*** 15.8 mm to (164.8, 87.8)
- moved C23 13.4 mm to (183.5, 157.5), turned to -90 degrees
- moved C22 9.52 mm to (186.0, 150.5), turned to -90 degrees
- moved FB13 9.00 mm to (183.5, 150.5)
- moved G*** 4.25 mm to (161.8, 92.0)
Connections:
- J1 pad 10: TUNE_OUT ??? -> GND
Routing:
- net TUNE_OUT ???: track 63.8 -> 0.00 mm, vias 2 -> 0
- net PTT_OUT: track 64.7 -> 49.9 mm, vias 2 -> 1
- net Net-(J12-Pin_1): track 18.9 -> 5.00 mm
- net Net-(J8-Pin_1): track 5.03 -> 0.00 mm
- net Net-(J8-Pin_2): track 5.00 -> 0.00 mm
- net Net-(J3-Pin_2): track 3.95 -> 0.00 mm
- net R_LINE_IN: track 93.4 -> 92.3 mm
- net GND: vias 33 -> 63
Other:
- board text added: "F6ITU 08/2023 https://github.com/F6ITU/K_IO_Board"
- board text added: "To Headset Andromeda J5 (Audio I/O)"
- board text removed: "External ATU"
- board text removed: "Internal ATU"
- board text removed: "To Headset Andromeda J5"
