File: K_IO_brd.kicad_sch (KiCad schematic)
At the start: 103 parts, among them J1 Conn from SDR J1, J10 To Andromeda J7, J11 PTT Out, J12 PTT Int, J13 SPKR Mute, J14 Jack_in/out, J15 to Andromeda J2, J18 Conn_01x02_Socket, J19 To SDR, J2 ACC Out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

Commit message: minor changes
Parts:
- removed C16, C21, C24, C25, C27: 10n, Capacitor_SMD:C_0805_2012Metric_Pad1.18x1.45mm_HandSolder, symbol Device:C_Small
- removed FB12, FB14, FB15: fb0805, Inductor_SMD:L_0805_2012Metric_Pad1.15x1.40mm_HandSolder, symbol Device:FerriteBead_Small
- removed J3: ATU Int, Connector_Molex:Molex_KK-254_AE-6410-03A_1x03_P2.54mm_Vertical, symbol Connector_Generic:Conn_01x03
- removed J8: Tune Ext ATU, Connector_Molex:Molex_KK-254_AE-6410-04A_1x04_P2.54mm_Vertical, symbol Connector_Generic:Conn_01x04
Connections:
- net TUNE_OUT ??? is gone; now on net GND: J1.10 (Pin_10)
- no-connect marks 18 -> 16
Other:
- moved on the sheet: J12
